File: kicad/m3/v1.1/TRSIO.kicad_pcb (KiCad board)
At the start: 2 copper layers, 93.3 x 72 mm, 28 parts, among them J1 TRS80, J2 +5V, J3 BUTTON, J4 LED, J5 FreHD Disable, Q1 2N7000, Q2 2N7000, Q3 2N7000, SW1 SW_Push, SW2 Right Angle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

Commit message: Updated M3 for compatibility with Kicad 5.1.5
Connections:
- J1 pad 37: (no net) -> //RESET
- J1 pad 45: (no net) -> /NC
- J1 pad 47: (no net) -> //M1
- U1A1 pad 10: (no net) -> Net-(U1A1-Pad10)
- U1A1 pad 16: (no net) -> Net-(U1A1-Pad16)
- U1A1 pad 17: (no net) -> Net-(U1A1-Pad17)
- U1A1 pad 18: (no net) -> Net-(U1A1-Pad18)
- U1A1 pad 2: (no net) -> Net-(U1A1-Pad2)
- U1A1 pad 20: (no net) -> Net-(U1A1-Pad20)
- U1A1 pad 21: (no net) -> Net-(U1A1-Pad21)
- U1A1 pad 22: (no net) -> Net-(U1A1-Pad22)
- U1A1 pad 24: (no net) -> Net-(U1A1-Pad24)
- U1A1 pad 25: (no net) -> Net-(U1A1-Pad25)
- U1A1 pad 34: (no net) -> Net-(U1A1-Pad34)
- U1A1 pad 35: (no net) -> Net-(U1A1-Pad35)
- U1B1 pad 12: (no net) -> Net-(U1B1-Pad12)
- U1B1 pad 13: (no net) -> Net-(U1B1-Pad13)
- U1B1 pad 16: (no net) -> Net-(U1B1-Pad16)
- U1B1 pad 24: (no net) -> Net-(U1B1-Pad24)
- U1B1 pad 4: (no net) -> Net-(U1B1-Pad4)
- U3 pad 11: (no net) -> Net-(U3-Pad11)
- U4 pad 11: (no net) -> Net-(U4-Pad11)
