File: kicad/m3/v1.1/TRSIO.sch (KiCad schematic (older format))
At the start: 24 parts, among them J1 TRS80, J2 +5V, J3 BUTTON, J4 LED, J5 FreHD Disable, Q1 2N7000, Q2 2N7000, Q3 2N7000, SW1 SW_Push, SW2 Right Angle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

Commit message: Updated M3 for compatibility with Kicad 5.1.5
Parts:
- C1, C2, C3, C4: symbol C_Small -> Device:C_Small
- D1: symbol LED_RCBG -> Device:LED_RCBG
- J1: symbol Conn_02x25_Odd_Even -> conn:Conn_02x25_Odd_Even
- J2, J3, J5: symbol Conn_01x02 -> conn:Conn_01x02
- J4: symbol Conn_01x04 -> conn:Conn_01x04
- Q1, Q2, Q3: symbol 2N7000 -> transistors:2N7000
- R1, R2, R3, R4: symbol R -> Device:R
- SW1, SW2: symbol SW_Push -> switches:SW_Push
- U1A1: symbol ESP32S -> HiLetgoESP32s:ESP32S
- U1B1: symbol ESP32S_AliExpress -> HiLetgoESP32s:ESP32S_AliExpress
- U2, U4: symbol 74LS245 -> TRSIO-rescue:74LS245
- U3: symbol GAL16V8 -> TRSIO:GAL16V8
