File: kicad/m3/v1.2/TRSIO.kicad_pcb (KiCad board)
At the start: 2 copper layers, 93.3 x 80.6 mm, 29 parts, among them J1 TRS80, J2 +5V, J3 BUTTON, J4 LED, J5 FreHD Disable, J6 TRS80, Q1 2N7000, Q2 2N7000, Q3 2N7000, SW1 SW_Push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

Commit message: TRS-IO-M3 PCB v1.2 + SD Card + PCB Updates
1. Connect GND pins of the SD card to ground
2. SPI pins connected for ESP32S
3. Pullup for CS_SD
4. PCB Layout
Parts:
- removed the REF** at (214.6, 73.7)
- removed the REF** at (214.6, 135.9)
- removed the REF** at (130.8, 135.9)
- removed the REF** at (130.8, 73.7)
- added J7: SD_Card, TRSIO:TFP09-2-12B, B.Cu at (214.4, 96.9)
- added R10: 10K, Resistors_THT:R_Axial_DIN0207_L6.3mm_D2.5mm_P7.62mm_Horizontal, F.Cu at (154.8, 82.2)
- added R11: 10K, Resistors_THT:R_Axial_DIN0207_L6.3mm_D2.5mm_P7.62mm_Horizontal, F.Cu at (187.3, 81.1)
- added R5: 10K, Resistors_THT:R_Axial_DIN0207_L6.3mm_D2.5mm_P7.62mm_Horizontal, F.Cu at (189.8, 105.0)
- added R6: 10K, Resistors_THT:R_Axial_DIN0207_L6.3mm_D2.5mm_P7.62mm_Horizontal, F.Cu at (154.8, 89.5)
- added R7: 10K, Resistors_THT:R_Axial_DIN0207_L6.3mm_D2.5mm_P7.62mm_Horizontal, F.Cu at (154.8, 93.2)
- added R8: 10K, Resistors_THT:R_Axial_DIN0207_L6.3mm_D2.5mm_P7.62mm_Horizontal, F.Cu at (187.3, 92.1)
- added R9: 10K, Resistors_THT:R_Axial_DIN0207_L6.3mm_D2.5mm_P7.62mm_Horizontal, F.Cu at (154.8, 85.9)
- added REF**: MountingHole_2.2mm_M2, Mounting_Holes:MountingHole_2.2mm_M2, F.Cu at (214.4, 99.9)
- added REF**: MountingHole_2.2mm_M2, Mounting_Holes:MountingHole_2.2mm_M2, F.Cu at (214.2, 92.1)
- added U5: MCP23S08, Housings_DIP:DIP-18_W7.62mm, F.Cu at (193.0, 116.1)
- moved D1 22.0 mm to (211.6, 79.3)
- moved C3 4.27 mm to (188.3, 114.3)
- moved R1 1.21 mm to (174.6, 84.9)
- moved R2 1.02 mm to (174.6, 88.5)
- moved R3 0.64 mm to (174.6, 92.1)
Connections:
- U1A1 pad 10: Net-(U1A1-Pad10) -> (no net)
- U1A1 pad 12: ESP32_D2 -> SCK
- U1A1 pad 13: ESP32_D0 -> MISO
- U1A1 pad 15: ESP32_D1 -> MOSI
- U1A1 pad 16: Net-(U1A1-Pad16) -> (no net)
- U1A1 pad 17: Net-(U1A1-Pad17) -> (no net)
- U1A1 pad 18: Net-(U1A1-Pad18) -> (no net)
- U1A1 pad 2: Net-(U1A1-Pad2) -> (no net)
- U1A1 pad 20: Net-(U1A1-Pad20) -> (no net)
- U1A1 pad 21: Net-(U1A1-Pad21) -> (no net)
- U1A1 pad 22: Net-(U1A1-Pad22) -> (no net)
- U1A1 pad 23: ESP32_D3 -> CS_EXPAND
- U1A1 pad 24: Net-(U1A1-Pad24) -> (no net)
- U1A1 pad 25: Net-(U1A1-Pad25) -> (no net)
- U1A1 pad 27: ESP32_D4 -> CS_SD
- U1A1 pad 28: ESP32_D5 -> (no net)
- U1A1 pad 30: ESP32_D6 -> (no net)
- U1A1 pad 31: ESP32_D7 -> (no net)
- U1A1 pad 34: Net-(U1A1-Pad34) -> (no net)
- U1A1 pad 35: Net-(U1A1-Pad35) -> (no net)
- U1B1 pad 10: ESP32_D7 -> (no net)
- U1B1 pad 12: Net-(U1B1-Pad12) -> (no net)
- U1B1 pad 13: Net-(U1B1-Pad13) -> (no net)
- U1B1 pad 16: Net-(U1B1-Pad16) -> (no net)
- U1B1 pad 24: Net-(U1B1-Pad24) -> (no net)
- U1B1 pad 26: ESP32_D2 -> SCK
- U1B1 pad 27: ESP32_D0 -> MISO
- U1B1 pad 28: ESP32_D1 -> MOSI
- U1B1 pad 3: ESP32_D3 -> CS_EXPAND
- U1B1 pad 4: Net-(U1B1-Pad4) -> (no net)
- U1B1 pad 6: ESP32_D4 -> CS_SD
- U1B1 pad 7: ESP32_D5 -> (no net)
- U1B1 pad 9: ESP32_D6 -> (no net)
- U3 pad 11: Net-(U3-Pad11) -> (no net)
- U4 pad 11: Net-(U4-Pad11) -> (no net)
Routing:
- net MISO: track 0.00 -> 108.3 mm, vias 0 -> 1
- net MOSI: track 0.00 -> 85.7 mm, vias 0 -> 1
- net CS_EXPAND: track 0.00 -> 72.7 mm, vias 0 -> 4
- net SCK: track 0.00 -> 66.8 mm, vias 0 -> 2
- net ESP32_D6: track 75.9 -> 11.4 mm, vias 2 -> 0
- net ESP32_D7: track 75.7 -> 11.6 mm, vias 2 -> 0
- net ESP32_D3: track 73.9 -> 11.4 mm, vias 3 -> 0
- net ESP32_D5: track 73.4 -> 11.4 mm, vias 2 -> 0
- net ESP32_D4: track 73.4 -> 11.4 mm, vias 2 -> 0
- net Net-(J7-Pad1): track 0.00 -> 53.8 mm, vias 0 -> 2
- net CS_SD: track 0.00 -> 50.8 mm, vias 0 -> 2
- net Net-(J7-Pad8): track 0.00 -> 49.6 mm
- net +3V3: track 138.6 -> 185.4 mm, vias 3 -> 5
- net ESP32_D0: track 54.5 -> 11.4 mm, vias 2 -> 0
- net ESP32_D2: track 52.2 -> 11.4 mm, vias 2 -> 0
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
Commit message: TRS-IO-M3 PCB v1.2 + SD Card + PCB Updates
1. Updated labels for buffered data bus signals from ESP32_Dx to BDx.
2. Updated meta data on schematic and PCB
3. Added M3 mounting holes to PCB
Parts:
- removed the REF** at (214.4, 99.9)
- removed the REF** at (214.2, 92.1)
- added REF**: MountingHole_3.2mm_M3, Mounting_Holes:MountingHole_3.2mm_M3, F.Cu at (215.5, 137.4)
- added REF**: MountingHole_3.2mm_M3, Mounting_Holes:MountingHole_3.2mm_M3, F.Cu at (129.3, 137.4)
- added REF**: MountingHole_3.2mm_M3, Mounting_Holes:MountingHole_3.2mm_M3, F.Cu at (215.5, 72.5)
- added REF**: MountingHole_3.2mm_M3, Mounting_Holes:MountingHole_3.2mm_M3, F.Cu at (129.3, 72.5)
Connections:
- net ESP32_D0 renamed BD0
- net ESP32_D1 renamed BD1
- net ESP32_D2 renamed BD2
- net ESP32_D3 renamed BD3
- net ESP32_D4 renamed BD4
- net ESP32_D5 renamed BD5
- net ESP32_D6 renamed BD6
- net ESP32_D7 renamed BD7
Other:
- board text added: "Updated TRS-IO with SD Card Support and Edge Connector"
- board text removed: "Reconfiguration of RetroStoreCard to support TRS-HD Emulation Prepared by Andrew Quinn"

Commit message: TRS-IO-M3 PCB v1.2 + SD Card + PCB Updates
1.  Added pin number labels to the edge connector.
2.  Added alignment holes below the SD Card.
Parts:
- added REF**: MountingHole_2.2mm_M2, Mounting_Holes:MountingHole_2.2mm_M2, F.Cu at (214.4, 100.0)
- added REF**: MountingHole_2.2mm_M2, Mounting_Holes:MountingHole_2.2mm_M2, F.Cu at (214.4, 92.1)
Other:
- board text added: "1"
- board text added: "2"
- board text added: "49"
- board text added: "50"
Changed lines of the file:
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@@
   (general
     (thickness 1.6)
-    (drawings 19)
+    (drawings 23)
     (tracks 746)
     (zones 0)
-    (modules 38)
+    (modules 40)
     (nets 66)
   )
@@
     (mod_text_size 1 1)
     (mod_text_width 0.15)
-    (pad_size 1.524 1.524)
-    (pad_drill 0.762)
+    (pad_size 2.2 2.2)
+    (pad_drill 2.2)
     (pad_to_mask_clearance 0.2)
     (aux_axis_origin 0 0)
@@
     (add_net _RESET)
   )
+  (module Mounting_Holes:MountingHole_2.2mm_M2 (layer F.Cu)
+    (at 214.376 100.0125)
+    (descr "Mounting Hole 2.2mm, no annular, M2")
+    (tags "mounting hole 2.2mm no annular m2")
+    (attr virtual)
+    (fp_text reference REF** (at 0 -3.2) (layer F.SilkS) hide
+      (effects (font (size 1 1) (thickness 0.15)))
+    )
+    (fp_text value MountingHole_2.2mm_M2 (at 0 3.2) (layer F.Fab)
+      (effects (font (size 1 1) (thickness 0.15)))
+    )
+    (fp_circle (center 0 0) (end 2.45 0) (layer F.CrtYd) (width 0.05))
+    (fp_circle (center 0 0) (end 2.2 0) (layer Cmts.User) (width 0.15))
+    (fp_text user %R (at 0.3 0) (layer F.Fab)
+      (effects (font (size 1 1) (thickness 0.15)))
+    )
+    (pad 1 np_thru_hole circle (at 0 0) (size 2.2 2.2) (drill 2.2) (layers *.Cu *.Mask))
+  )
+  (module Mounting_Holes:MountingHole_2.2mm_M2 (layer F.Cu)
+    (at 214.376 92.075)
+    (descr "Mounting Hole 2.2mm, no annular, M2")
+    (tags "mounting hole 2.2mm no annular m2")
+    (attr virtual)
+    (fp_text reference REF** (at 0 -3.2) (layer F.SilkS) hide
+      (effects (font (size 1 1) (thickness 0.15)))
+    )
+    (fp_text value MountingHole_2.2mm_M2 (at 0 3.2) (layer F.Fab)
+      (effects (font (size 1 1) (thickness 0.15)))
+    )
+    (fp_text user %R (at 0.3 0) (layer F.Fab)
+      (effects (font (size 1 1) (thickness 0.15)))
+    )
+    (fp_circle (center 0 0) (end 2.2 0) (layer Cmts.User) (width 0.15))
+    (fp_circle (center 0 0) (end 2.45 0) (layer F.CrtYd) (width 0.05))
+    (pad 1 np_thru_hole circle (at 0 0) (size 2.2 2.2) (drill 2.2) (layers *.Cu *.Mask))
+  )
   (module Mounting_Holes:MountingHole_3.2mm_M3 (layer F.Cu)
     (at 215.519 137.414)
@@
     )
   )
-  (gr_text "TRS-IO V1.2\nAugust 2021" (at 214.63 91.44) (layer F.SilkS)
+  (gr_text 50 (at 139.5095 140.0175) (layer B.SilkS)
+    (effects (font (size 1 1) (thickness 0.15)) (justify mirror))
+  )
+  (gr_text 2 (at 202.946 140.0175) (layer B.SilkS)
+    (effects (font (size 1 1) (thickness 0.15)) (justify mirror))
+  )
+  (gr_text 49 (at 139.5095 140.0175) (layer F.SilkS)
+    (effects (font (size 1 1) (thickness 0.15)))
+  )
+  (gr_text 1 (at 202.946 140.0175) (layer F.SilkS)
+    (effects (font (size 1 1) (thickness 0.15)))
+  )
+  (gr_text "TRS-IO V1.2\nAugust 2021" (at 214.63 87.503) (layer F.SilkS)
     (effects (font (size 1.5 1.5) (thickness 0.3)) (justify right))
   )
