File: kicad/m1/v1.2-xray/TRS-IO-M1.kicad_sch (KiCad schematic)
At the start: 32 parts, among them J1 Conn_02x20_Odd_Even, J2 Conn_02x20_Odd_Even, J3 SD_Card, J4 Conn_01x02_Male, J5 Conn_01x02_Male, Q1 2N7000, Q2 2N7000, SW1 SW_Push, U1 HiLetgo-ESP-32S, U2 Artix-7-15T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

Commit message: Add VGA to TRS-IO-XRAY schematics and PCB
Parts:
- added J6: DB15_Female_HighDensity, TRS-IO-M1:DB_15F-VGA, symbol Connector:DB15_Female_HighDensity
- added U7: MCP43x1, Package_SO:TSSOP-20_4.4x6.5mm_P0.65mm, symbol MCP43X1:MCP43x1
- H1, H2, H3, H4: footprint MountingHole:MountingHole_2.5mm_Pad_Via -> MountingHole:MountingHole_3mm_Pad_Via
Connections:
- net +3V3: now also U7.17 (VDD)
- net AA0: now also U2.26 (pio26); no longer U2.1 (pio1)
- net AA1: now also U2.23 (pio23); no longer U2.48 (pio48)
- net AA10: now also U2.30 (pio30); no longer U2.5 (pio5)
- net AA11: now also U2.19 (pio19); no longer U2.44 (pio44)
- net AA12: now also U2.31 (pio31); no longer U2.6 (pio6)
- net AA13: now also U2.32 (pio32); no longer U2.7 (pio7)
- net AA14: now also U2.18 (pio18); no longer U2.43 (pio43)
- net AA15: now also U2.33 (pio33); no longer U2.8 (pio8)
- net AA2: now also U2.20 (pio20); no longer U2.45 (pio45)
- net AA3: now also U2.22 (pio22); no longer U2.47 (pio47)
- net AA4: now also U2.27 (pio27); no longer U2.2 (pio2)
- net AA5: now also U2.28 (pio28); no longer U2.3 (pio3)
- net AA6: now also U2.29 (pio29); no longer U2.4 (pio4)
- net AA7: now also U2.21 (pio21); no longer U2.46 (pio46)
- net AA8: now also U2.17 (pio17); no longer U2.42 (pio42)
- net AA9: now also U2.14 (pio14); no longer U2.41 (pio41)
- net CS_FPGA: now also U2.5 (pio5); no longer U2.32 (pio32)
- net DBUS_SEL_N: now also U2.48 (pio48); no longer U2.29 (pio29)
- net DD0: now also U2.40 (pio40); no longer U2.17 (pio17)
- net DD1: now also U2.36 (pio36); no longer U2.11 (pio11)
- net DD2: now also U2.41 (pio41); no longer U2.18 (pio18)
- net DD3: now also U2.38 (pio38); no longer U2.13 (pio13)
- net DD4: now also U2.34 (pio34); no longer U2.9 (pio9)
- net DD5: now also U2.39 (pio39); no longer U2.14 (pio14)
- net DD6: now also U2.37 (pio37); no longer U2.12 (pio12)
- net DD7: now also U2.35 (pio35); no longer U2.10 (pio10)
- net DONE: now also U2.13 (pio13); no longer U2.40 (pio40)
- net ESP_S0: now also U2.11 (pio11); no longer U2.38 (pio38)
- net ESP_S1: now also U2.10 (pio10); no longer U2.37 (pio37)
- net ESP_S2: now also U2.9 (pio9); no longer U2.36 (pio36)
- net FULL_ADDR: now also U1.27 (GPIO33); no longer U2.30 (pio30)
- net GND: now also J6.10, J6.5, J6.6, J6.7, J6.8, U7.13 (P0B), U7.18 (P2B), U7.7 (VSS), U7.8 (P1B)
- net INT: now also U2.1 (pio1); no longer U2.26 (pio26)
- net MISO: now also U2.6 (pio6), U7.16 (SDO); no longer U2.33 (pio33)
- net MOSI: now also U2.7 (pio7), U7.6 (SDI); no longer U2.34 (pio34)
- net READ_N: now also U2.47 (pio47); no longer U2.28 (pio28)
- net REQ: now also U2.12 (pio12); no longer U2.39 (pio39)
- net SCK: now also U2.4 (pio4), U7.5 (SCK); no longer U2.31 (pio31)
- net WAIT: now also U2.46 (pio46); no longer U2.27 (pio27)
- net Z80_IN_N: now also U2.45 (pio45); no longer U2.23 (pio23)
- net Z80_OUT_N: now also U2.44 (pio44); no longer U2.22 (pio22)
- net Z80_RAS_N: no longer U2.21 (pio21)
- net Z80_RD_N: now also U2.43 (pio43); no longer U2.20 (pio20)
- net Z80_WR_N: now also U2.42 (pio42); no longer U2.19 (pio19)
- net ESP_S3 renamed CS_MCP43x1
- net CS_MCP43x1: now also U7.4 (~{CS}); no longer U2.35 (pio35)
- new net POT_VGA_BLUE: J6.3, U7.19 (P2W)
- new net POT_VGA_GREEN: J6.2, U7.9 (P1W)
- new net POT_VGA_RED: J6.1, U7.12 (P0W)
- new net VGA_HSYNC: J6.13, U2.3 (pio3)
- new net VGA_RGB: U2.8 (pio8), U7.10 (P1A), U7.11 (P0A), U7.20 (P2A)
- new net VGA_VSYNC: J6.14, U2.2 (pio2)
Other:
- moved on the sheet: D1, H1, H2, H3, H4, J3, J4, J5, Q1, Q2, R1, R2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
