File: kicad/pp/v0.2/TRS-IO++.kicad_pcb (KiCad board)
At the start: 2 copper layers, 145.7 x 107.8 mm, 99 parts, among them J1 TRS-80 M3 Pin Header, J10 AudioJack3, J11 Mini-DIN-6, J12 USB_B_Micro, J2 TRS-80 M1 Pin Connector, J3 TRS-80 M3 Edge Connector, J4 TRS-80 M1 Edge Connector, J5 Conn_01x06_Male, J6 Conn_01x06_Male, J7 HDMI_A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

Commit message: Move diagnostic LEDs to PCB edge
Parts:
- moved R37 5.23 mm to (46.8, 138.5)
- moved R38 5.23 mm to (49.9, 138.5)
- moved R39 5.23 mm to (52.9, 138.5)
- moved R40 5.23 mm to (56.0, 138.5)
- moved D2 5.23 mm to (46.8, 143.8)
- moved D3 5.23 mm to (49.8, 143.8)
- moved D4 5.23 mm to (52.9, 143.8)
- moved D5 5.23 mm to (55.9, 143.8)
Connections:
- D2 pad 1: Net-(D2-Pad1) -> GND
- D2 pad 2: LED1 -> Net-(D2-Pad2)
- D3 pad 1: Net-(D3-Pad1) -> GND
- D3 pad 2: LED2 -> Net-(D3-Pad2)
- D4 pad 1: Net-(D4-Pad1) -> GND
- D4 pad 2: LED3 -> Net-(D4-Pad2)
- D5 pad 1: Net-(D5-Pad1) -> GND
- D5 pad 2: LED4 -> Net-(D5-Pad2)
- R37 pad 1: Net-(D2-Pad1) -> LED1
- R37 pad 2: GND -> Net-(D2-Pad2)
- R38 pad 1: Net-(D3-Pad1) -> LED2
- R38 pad 2: GND -> Net-(D3-Pad2)
- R39 pad 1: Net-(D4-Pad1) -> LED3
- R39 pad 2: GND -> Net-(D4-Pad2)
- R40 pad 1: Net-(D5-Pad1) -> LED4
- R40 pad 2: GND -> Net-(D5-Pad2)
Routing:
- net Net-(D4-Pad2): track 0.00 -> 3.19 mm
- net Net-(D4-Pad1): track 3.19 -> 0.00 mm
- net Net-(D3-Pad2): track 0.00 -> 3.19 mm
- net Net-(D3-Pad1): track 3.19 -> 0.00 mm
- net Net-(D5-Pad2): track 0.00 -> 3.16 mm
- net Net-(D5-Pad1): track 3.16 -> 0.00 mm
- net Net-(D2-Pad2): track 0.00 -> 3.16 mm
- net Net-(D2-Pad1): track 3.16 -> 0.00 mm
Other:
- board text added: "TRS-IO++ V0.2 February 2023"
- board text removed: "TRS-IO++ V0.2 January 2023"

Commit message: Route JTAG TDI/TDO to different GPIOs
Connections:
- Conn1 pad 147: RXD0 -> JTAG_TDO
- Conn1 pad 153: TXD0 -> JTAG_TDI
- U1 pad 12: unconnected-(U1-Pad12) -> JTAG_TDO
- U1 pad 5: unconnected-(U1-Pad5) -> JTAG_TDI
Routing:
- net TXD0: track 163.4 -> 37.5 mm, vias 2 -> 0
- net RXD0: track 155.8 -> 33.8 mm, vias 2 -> 0
- net JTAG_TDI: track 0.00 -> 110.4 mm, vias 0 -> 2
- net JTAG_TDO: track 0.00 -> 99.4 mm, vias 0 -> 2
- net JTAG_TCK: track 126.8 -> 126.2 mm
